Commit message: zed camera updates

File: description/robot.urdf.xacro (robot description, xacro)
@@ -5,5 +5,5 @@
   <xacro:arg name="camera_model"  default="zed2" />
   <xacro:arg name="use_zed_localization" default="true" />
-  <xacro:arg name="baseline" default="0.0" />
+  <xacro:arg name="baseline" default="-0.1" />
   <xacro:arg name="enable_gnss" default="false" />
   <xacro:include filename="$(find shimmy_bot)/description/robot_description.urdf.xacro" />
@@ -13,5 +13,5 @@
   <xacro:diffbot/>
 <xacro:property name="depth_sensor_pose">
-    <origin xyz="0.14 0.0 0.045" rpy="0 0 0"/>
+    <origin xyz="0.14 0.0 0.5" rpy="1.5708 0 0"/>
 </xacro:property>
 <!--
@@ -21,5 +21,5 @@
   <xacro:diffbot_ros2_control
     name="DiffBot" use_mock_hardware="$(arg use_mock_hardware)"/>
-  <xacro:include filename="$(find shimmy_bot)/description/zed_macro.urdf.xacro" />
+  <xacro:include filename="$(find zed_wrapper)/urdf/zed_macro.urdf.xacro" />
   <xacro:zed_camera name="$(arg camera_name)" model="$(arg camera_model)">
   <xacro:insert_block name="depth_sensor_pose" />
@@ -29,5 +29,5 @@
       <child link="base_link"/>
       <origin
-        xyz="-0.012 0.0 -0.25"
+        xyz="-0.0 0.0 0.12"
         rpy="0 0 0"
       />

File: description/zed_macro.urdf.xacro (robot description, xacro)
@@ -44,7 +44,7 @@
       <xacro:property name="baseline" value="0.12" />
       <xacro:property name="height" value="0.03" />
-      <xacro:property name="bottom_slope" value="0.05" />
+      <xacro:property name="bottom_slope" value="0.00" />
       <xacro:property name="screw_offset_x" value="0.0" />
-      <xacro:property name="screw_offset_z" value="0.0" />
+      <xacro:property name="screw_offset_z" value="0.473" />
       <xacro:property name="optical_offset_x" value="-0.01" />
     </xacro:if>
@@ -79,5 +79,5 @@
       <xacro:unless value="${model == 'virtual'}">
         <visual>
-          <origin xyz="${screw_offset_x} 0 ${screw_offset_z}" rpy="0 0 0"/>
+          <origin xyz="${screw_offset_x} 0 ${screw_offset_z}" rpy="1.5708 0 0"/>
           <geometry>
             <mesh filename="package://zed_interfaces/meshes/${model}.stl" />
@@ -86,5 +86,5 @@
         </visual>
         <collision>
-          <origin xyz="${screw_offset_x} 0 ${screw_offset_z}" rpy="0 0 0"/>
+          <origin xyz="${screw_offset_x} 0 ${screw_offset_z}" rpy="1.5708 0 0"/>
           <geometry>
             <mesh filename="package://zed_interfaces/meshes/${model}.stl" />
@@ -96,5 +96,5 @@
       <parent link="${name}_camera_link"/>
       <child link="${name}_camera_center"/>
-      <origin xyz="0.10 0 0.350" rpy="0 ${bottom_slope} 0" />
+      <origin xyz="0.0 0.0 0.0" rpy="0 ${bottom_slope} 0" />
     </joint>
     <!-- Left Camera -->
@@ -123,5 +123,5 @@
     <link name="${name}_left_camera_optical_frame"/>
     <joint name="${name}_left_camera_optical_joint" type="fixed">
-      <origin xyz="0 0 0" rpy="-${M_PI/2} 0.0 -${M_PI/2}"/>
+      <origin xyz="0 0 0" rpy="0.0 0.0 0.0"/>
       <parent link="${name}_left_camera_frame"/>
       <child link="${name}_left_camera_optical_frame"/>
@@ -137,5 +137,5 @@
     <link name="${name}_right_camera_optical_frame"/>
     <joint name="${name}_right_camera_optical_joint" type="fixed">
-      <origin xyz="0 0 0" rpy="-${M_PI/2} 0.0 -${M_PI/2}"/>
+      <origin xyz="0 0 0" rpy="0.0 0.0 0.0"/>
       <parent link="${name}_right_camera_frame"/>
       <child link="${name}_right_camera_optical_frame"/>

Commit message: nav2 updates

File: description/robot.urdf.xacro (robot description, xacro)
@@ -21,5 +21,5 @@
   <xacro:diffbot_ros2_control
     name="DiffBot" use_mock_hardware="$(arg use_mock_hardware)"/>
-  <xacro:include filename="$(find zed_wrapper)/urdf/zed_macro.urdf.xacro" />
+  <xacro:include filename="$(find shimmy_bot)/description/zed_macro.urdf.xacro" />
   <xacro:zed_camera name="$(arg camera_name)" model="$(arg camera_model)">
   <xacro:insert_block name="depth_sensor_pose" />

File: description/zed_macro.urdf.xacro (robot description, xacro)
@@ -24,5 +24,5 @@
       - enable_gnss: if true enable the URDF link
   -->
-  <xacro:macro name="zed_camera" params="name=zed model=zed enable_gnss=false custom_baseline=0 *origin">
+  <xacro:macro name="zed_camera" params="name=zed model=zed enable_gnss=false custom_baseline=0 *gnss_origin">
     <xacro:if value="${model == 'zed'}">
       <xacro:property name="baseline" value="0.12" />
@@ -44,7 +44,7 @@
       <xacro:property name="baseline" value="0.12" />
       <xacro:property name="height" value="0.03" />
-      <xacro:property name="bottom_slope" value="0.00" />
-      <xacro:property name="screw_offset_x" value="0.0" />
-      <xacro:property name="screw_offset_z" value="0.473" />
+      <xacro:property name="bottom_slope" value="0.05" />
+      <xacro:property name="screw_offset_x" value="0.0" />
+      <xacro:property name="screw_offset_z" value="0.46" />
       <xacro:property name="optical_offset_x" value="-0.01" />
     </xacro:if>
@@ -72,4 +72,12 @@
       <xacro:property name="screw_offset_z" value="-0.016" />
       <xacro:property name="optical_offset_x" value="-0.01" />
+    </xacro:if>
+    <xacro:if value="${model == 'virtual'}">
+      <xacro:property name="baseline" value="${custom_baseline}" />
+      <xacro:property name="height" value="0.031" />
+      <xacro:property name="bottom_slope" value="0.0" />
+      <xacro:property name="screw_offset_x" value="0.00" />
+      <xacro:property name="screw_offset_z" value="-0.0155" />
+      <xacro:property name="optical_offset_x" value="0.0" />
     </xacro:if>
     <!-- Camera mounting point (the threaded screw hole in the bottom) -->
@@ -79,5 +87,5 @@
       <xacro:unless value="${model == 'virtual'}">
         <visual>
-          <origin xyz="${screw_offset_x} 0 ${screw_offset_z}" rpy="1.5708 0 0"/>
+          <origin xyz="${screw_offset_x} 0 ${screw_offset_z}" rpy="0 0 0"/>
           <geometry>
             <mesh filename="package://zed_interfaces/meshes/${model}.stl" />
@@ -86,5 +94,5 @@
         </visual>
         <collision>
-          <origin xyz="${screw_offset_x} 0 ${screw_offset_z}" rpy="1.5708 0 0"/>
+          <origin xyz="${screw_offset_x} 0 ${screw_offset_z}" rpy="0 0 0"/>
           <geometry>
             <mesh filename="package://zed_interfaces/meshes/${model}.stl" />
@@ -96,5 +104,5 @@
       <parent link="${name}_camera_link"/>
       <child link="${name}_camera_center"/>
-      <origin xyz="0.0 0.0 0.0" rpy="0 ${bottom_slope} 0" />
+      <origin xyz="0 0 ${height/2}" rpy="0 ${bottom_slope} 0" />
     </joint>
     <!-- Left Camera -->
@@ -123,5 +131,5 @@
     <link name="${name}_left_camera_optical_frame"/>
     <joint name="${name}_left_camera_optical_joint" type="fixed">
-      <origin xyz="0 0 0" rpy="0.0 0.0 0.0"/>
+      <origin xyz="0 0 0" rpy="-${M_PI/2} 0.0 -${M_PI/2}"/>
       <parent link="${name}_left_camera_frame"/>
       <child link="${name}_left_camera_optical_frame"/>
@@ -129,4 +137,19 @@
     <!-- Right Camera -->
     <link name="${name}_right_camera_frame">
+      <xacro:if value="${model == 'virtual'}">
+        <visual>
+          <origin xyz="0 0 0" rpy="0 0 0"/>
+          <geometry>
+            <mesh filename="package://zed_interfaces/meshes/${model}.stl" />
+          </geometry>
+          <material name="${model}_mat" />
+        </visual>
+        <collision>
+          <origin xyz="0 0 0" rpy="0 0 0"/>
+          <geometry>
+            <mesh filename="package://zed_interfaces/meshes/${model}.stl" />
+          </geometry>
+        </collision>
+      </xacro:if>
     </link>
     <joint name="${name}_right_camera_joint" type="fixed">
@@ -137,5 +160,5 @@
     <link name="${name}_right_camera_optical_frame"/>
     <joint name="${name}_right_camera_optical_joint" type="fixed">
-      <origin xyz="0 0 0" rpy="0.0 0.0 0.0"/>
+      <origin xyz="0 0 0" rpy="-${M_PI/2} 0.0 -${M_PI/2}"/>
       <parent link="${name}_right_camera_frame"/>
       <child link="${name}_right_camera_optical_frame"/>

Commit message: general updates

File: description/robot.urdf.xacro (robot description, xacro)
@@ -5,23 +5,20 @@
   <xacro:arg name="camera_model"  default="zed2" />
   <xacro:arg name="use_zed_localization" default="true" />
-  <xacro:arg name="baseline" default="-0.1" />
+  <xacro:arg name="baseline" default="0.0" />
   <xacro:arg name="enable_gnss" default="false" />
   <xacro:include filename="$(find shimmy_bot)/description/robot_description.urdf.xacro" />
   <xacro:include filename="$(find shimmy_bot)/description/robot.ros2_control.xacro" />
-  <!-- <xacro:include filename="$(find shimmy_bot)/description/depth_sensor.urdf.xacro" /> -->
-  <!-- Add one ZED Camera -->
+  <!-- <xacro:include filename="$(find shimmy_bot)/description/d435.urdf.xacro" /> -->
+  <xacro:diffbot_ros2_control name="DiffBot" use_mock_hardware="$(arg use_mock_hardware)"/>
   <xacro:diffbot/>
-<xacro:property name="depth_sensor_pose">
+  <xacro:property name="depth_sensor_pose">
     <origin xyz="0.14 0.0 0.5" rpy="1.5708 0 0"/>
-</xacro:property>
-<!--
-  <xacro:depth_sensor>
-    <xacro:insert_block name="depth_sensor_pose" />
-  </xacro:depth_sensor> -->
-  <xacro:diffbot_ros2_control
-    name="DiffBot" use_mock_hardware="$(arg use_mock_hardware)"/>
+  </xacro:property>
+  <!-- <xacro:sensor_d435 name="camera" topics_ns="camera" parent="base_link" publish_pointcloud="true">
+    <origin xyz="0.02 0 0.44" rpy="0 0 0" />
+  </xacro:sensor_d435>   -->
   <xacro:include filename="$(find shimmy_bot)/description/zed_macro.urdf.xacro" />
   <xacro:zed_camera name="$(arg camera_name)" model="$(arg camera_model)">
-  <xacro:insert_block name="depth_sensor_pose" />
+    <xacro:insert_block name="depth_sensor_pose" />
   </xacro:zed_camera>
     <joint name="$(arg camera_name)_joint" type="fixed">
@@ -29,5 +26,5 @@
       <child link="base_link"/>
       <origin
-        xyz="-0.0 0.0 0.12"
+        xyz="-0.12 0.0 -0.35"
         rpy="0 0 0"
       />

File: description/robot_description.urdf.xacro (robot description, xacro)
@@ -13,5 +13,5 @@
   <xacro:property name="caster_wheel_mass" value="0.1" /> <!-- arbitrary value for caster wheel mass -->
   <xacro:property name="caster_wheel_radius" value="0.015" />
-  <xacro:property name="z_offset" value="-${base_height/2}" /> <!-- Space btw top of beam and the each joint -->
+  <xacro:property name="z_offset" value="0.050" /> <!-- Space btw top of beam and the each joint -->
   <xacro:property name="x_offset" value="0.075" />
   <xacro:property name="y_offset" value="0.150" />
@@ -46,5 +46,5 @@
     </collision>
     <visual>
-      <origin xyz="0 0 ${base_height/2}" rpy="0 0 0"/>
+      <origin xyz="0 0 0.185" rpy="0 0 0"/>
       <geometry>
         <box size="${base_width} ${base_length} ${base_height}"/>
@@ -162,5 +162,5 @@
       <parent link="base_link"/>
       <child link="speaker_link"/>
-      <origin xyz="-0.060 0  0.2375" rpy="0 0 0"/>
+      <origin xyz="-0.060 0  0.350" rpy="0 0 0"/>
     </joint>
     <link name="speaker_link">

File: description/zed_macro.urdf.xacro (robot description, xacro)
@@ -42,9 +42,9 @@
     </xacro:if>
     <xacro:if value="${model == 'zed2'}">
-      <xacro:property name="baseline" value="0.12" />
+      <xacro:property name="baseline" value="0.0" />
       <xacro:property name="height" value="0.03" />
       <xacro:property name="bottom_slope" value="0.05" />
-      <xacro:property name="screw_offset_x" value="0.0" />
-      <xacro:property name="screw_offset_z" value="0.46" />
+      <xacro:property name="screw_offset_x" value="-0.10" />
+      <xacro:property name="screw_offset_z" value="0.09" />
       <xacro:property name="optical_offset_x" value="-0.01" />
     </xacro:if>

Commit message: agent updates

File: description/robot.urdf.xacro (robot description, xacro)
@@ -23,8 +23,8 @@
   </xacro:zed_camera>
     <joint name="$(arg camera_name)_joint" type="fixed">
-      <parent link="$(arg camera_name)_camera_link"/>
-      <child link="base_link"/>
+      <parent link="base_link"/>
+      <child link="$(arg camera_name)_camera_link"/>
       <origin
-        xyz="-0.12 0.0 -0.35"
+        xyz="0.12 0.0 0.35"
         rpy="0 0 0"
       />
