Commit message: updates to navigation

File: description/robot.urdf.xacro (robot description, xacro)
@@ -12,7 +12,7 @@
   <xacro:diffbot_ros2_control name="DiffBot" use_mock_hardware="$(arg use_mock_hardware)"/>
   <xacro:diffbot/>
-  <xacro:property name="depth_sensor_pose">
+  <!-- <xacro:property name="depth_sensor_pose">
     <origin xyz="0.14 0.0 0.5" rpy="1.5708 0 0"/>
-  </xacro:property>
+  </xacro:property> -->
   <!-- <xacro:sensor_d435 name="camera" topics_ns="camera" parent="base_link" publish_pointcloud="true">
     <origin xyz="0.02 0 0.44" rpy="0 0 0" />
@@ -20,13 +20,13 @@
   <xacro:include filename="$(find shimmy_bot)/description/zed_macro.urdf.xacro" />
   <xacro:zed_camera name="$(arg camera_name)" model="$(arg camera_model)">
-    <xacro:insert_block name="depth_sensor_pose" />
   </xacro:zed_camera>
-    <joint name="$(arg camera_name)_joint" type="fixed">
-      <parent link="base_link"/>
-      <child link="$(arg camera_name)_camera_link"/>
-      <origin
-        xyz="0.12 0.0 0.35"
-        rpy="0 0 0"
-      />
-    </joint>
+  <!-- Add a joint to connect the ZED Camera to the robot -->
+  <joint name="$(arg camera_name)_joint" type="fixed">
+    <parent link="$(arg camera_name)_camera_link"/>
+    <child link="base_link"/>
+    <origin
+      xyz="-0.05 0.0 0.0"
+      rpy="0 0 0"
+    />
+  </joint>
 </robot>

File: description/zed_macro.urdf.xacro (robot description, xacro)
@@ -1,5 +1,5 @@
 <?xml version="1.0"?>
 <!--
-// Copyright 2022 Stereolabs
+// Copyright 2024 Stereolabs
 //
 // Licensed under the Apache License, Version 2.0 (the "License");
@@ -24,5 +24,5 @@
       - enable_gnss: if true enable the URDF link
   -->
-  <xacro:macro name="zed_camera" params="name=zed model=zed enable_gnss=false custom_baseline=0 *gnss_origin">
+  <xacro:macro name="zed_camera" params="name=zed model=zed enable_gnss=false custom_baseline=0">
     <xacro:if value="${model == 'zed'}">
       <xacro:property name="baseline" value="0.12" />
@@ -32,7 +32,8 @@
       <xacro:property name="screw_offset_z" value="0.0" />
       <xacro:property name="optical_offset_x" value="-0.01" />
+      <xacro:property name="mono" value="false" />
     </xacro:if>
     <xacro:if value="${model == 'zedm'}">
-      <xacro:property name="baseline" value="0.06" />
+      <xacro:property name="baseline" value="0.063" />
       <xacro:property name="height" value="0.0265" />
       <xacro:property name="bottom_slope" value="0.0" />
@@ -40,12 +41,14 @@
       <xacro:property name="screw_offset_z" value="0.0" />
       <xacro:property name="optical_offset_x" value="0.0" />
+      <xacro:property name="mono" value="false" />
     </xacro:if>
     <xacro:if value="${model == 'zed2'}">
-      <xacro:property name="baseline" value="0.0" />
+      <xacro:property name="baseline" value="0.12" />
       <xacro:property name="height" value="0.03" />
       <xacro:property name="bottom_slope" value="0.05" />
-      <xacro:property name="screw_offset_x" value="-0.10" />
-      <xacro:property name="screw_offset_z" value="0.09" />
-      <xacro:property name="optical_offset_x" value="-0.01" />
+      <xacro:property name="screw_offset_x" value="0.0" />
+      <xacro:property name="screw_offset_z" value="0.0" />
+      <xacro:property name="optical_offset_x" value="-0.01" />
+      <xacro:property name="mono" value="false" />
     </xacro:if>
     <xacro:if value="${model == 'zed2i'}">
@@ -56,4 +59,5 @@
       <xacro:property name="screw_offset_z" value="0.0" />
       <xacro:property name="optical_offset_x" value="-0.01" />
+      <xacro:property name="mono" value="false" />
     </xacro:if>
     <xacro:if value="${model == 'zedx'}">
@@ -64,4 +68,5 @@
       <xacro:property name="screw_offset_z" value="-0.016" />
       <xacro:property name="optical_offset_x" value="-0.01" />
+      <xacro:property name="mono" value="false" />
     </xacro:if>
     <xacro:if value="${model == 'zedxm'}">
@@ -72,4 +77,5 @@
       <xacro:property name="screw_offset_z" value="-0.016" />
       <xacro:property name="optical_offset_x" value="-0.01" />
+      <xacro:property name="mono" value="false" />
     </xacro:if>
     <xacro:if value="${model == 'virtual'}">
@@ -80,4 +86,23 @@
       <xacro:property name="screw_offset_z" value="-0.0155" />
       <xacro:property name="optical_offset_x" value="0.0" />
+      <xacro:property name="mono" value="false" />
+    </xacro:if>
+    <xacro:if value="${model == 'zedxonegs'}">
+      <xacro:property name="baseline" value="0.0" />
+      <xacro:property name="height" value="0.031" />
+      <xacro:property name="bottom_slope" value="0.0" />
+      <xacro:property name="screw_offset_x" value="0.0" />
+      <xacro:property name="screw_offset_z" value="-0.0155" />
+      <xacro:property name="optical_offset_x" value="0.0" />
+      <xacro:property name="mono" value="true" />
+    </xacro:if>
+    <xacro:if value="${model == 'zedxone4k'}">
+      <xacro:property name="baseline" value="0.0" />
+      <xacro:property name="height" value="0.031" />
+      <xacro:property name="bottom_slope" value="0.0" />
+      <xacro:property name="screw_offset_x" value="0.00" />
+      <xacro:property name="screw_offset_z" value="-0.0155" />
+      <xacro:property name="optical_offset_x" value="0.0" />
+      <xacro:property name="mono" value="true" />
     </xacro:if>
     <!-- Camera mounting point (the threaded screw hole in the bottom) -->
@@ -89,5 +114,5 @@
           <origin xyz="${screw_offset_x} 0 ${screw_offset_z}" rpy="0 0 0"/>
           <geometry>
-            <mesh filename="package://zed_interfaces/meshes/${model}.stl" />
+<mesh filename="file://$(find zed_msgs)/meshes/${model}.stl"/>
           </geometry>
           <material name="${model}_mat" />
@@ -96,5 +121,5 @@
           <origin xyz="${screw_offset_x} 0 ${screw_offset_z}" rpy="0 0 0"/>
           <geometry>
-            <mesh filename="package://zed_interfaces/meshes/${model}.stl" />
+<mesh filename="file://$(find zed_msgs)/meshes/${model}.stl"/>
           </geometry>
         </collision>
@@ -106,87 +131,104 @@
       <origin xyz="0 0 ${height/2}" rpy="0 ${bottom_slope} 0" />
     </joint>
-    <!-- Left Camera -->
-    <link name="${name}_left_camera_frame">
-      <xacro:if value="${model == 'virtual'}">
-        <visual>
-          <origin xyz="0 0 0" rpy="0 0 0"/>
-          <geometry>
-            <mesh filename="package://zed_interfaces/meshes/${model}.stl" />
-          </geometry>
-          <material name="${model}_mat" />
-        </visual>
-        <collision>
-          <origin xyz="0 0 0" rpy="0 0 0"/>
-          <geometry>
-            <mesh filename="package://zed_interfaces/meshes/${model}.stl" />
-          </geometry>
-        </collision>
+    <xacro:unless value="${mono}">
+      <!-- Left Camera -->
+      <link name="${name}_left_camera_frame">
+        <xacro:if value="${model == 'virtual'}">
+          <visual>
+            <origin xyz="0 0 0" rpy="0 0 0"/>
+            <geometry>
+  <mesh filename="file://$(find zed_msgs)/meshes/${model}.stl"/>
+            </geometry>
+            <material name="${model}_mat" />
+          </visual>
+          <collision>
+            <origin xyz="0 0 0" rpy="0 0 0"/>
+            <geometry>
+  <mesh filename="file://$(find zed_msgs)/meshes/${model}.stl"/>
+            </geometry>
+          </collision>
+        </xacro:if>
+      </link>
+      <joint name="${name}_left_camera_joint" type="fixed">
+        <parent link="${name}_camera_center"/>
+        <child link="${name}_left_camera_frame"/>
+        <origin xyz="${optical_offset_x} ${baseline/2} 0" rpy="0 0 0" />
+      </joint>
+      <link name="${name}_left_camera_optical_frame"/>
+      <joint name="${name}_left_camera_optical_joint" type="fixed">
+        <origin xyz="0 0 0" rpy="-${M_PI/2} 0.0 -${M_PI/2}"/>
+        <parent link="${name}_left_camera_frame"/>
+        <child link="${name}_left_camera_optical_frame"/>
+      </joint>
+      <!-- Right Camera -->
+      <link name="${name}_right_camera_frame">
+        <xacro:if value="${model == 'virtual'}">
+          <visual>
+            <origin xyz="0 0 0" rpy="0 0 0"/>
+            <geometry>
+  <mesh filename="file://$(find zed_msgs)/meshes/${model}.stl"/>
+            </geometry>
+            <material name="${model}_mat" />
+          </visual>
+          <collision>
+            <origin xyz="0 0 0" rpy="0 0 0"/>
+            <geometry>
+  <mesh filename="file://$(find zed_msgs)/meshes/${model}.stl"/>
+            </geometry>
+          </collision>
+        </xacro:if>
+      </link>
+      <joint name="${name}_right_camera_joint" type="fixed">
+        <parent link="${name}_camera_center"/>
+        <child link="${name}_right_camera_frame"/>
+        <origin xyz="${optical_offset_x} -${baseline/2} 0" rpy="0 0 0" />
+      </joint>
+      <link name="${name}_right_camera_optical_frame"/>
+      <joint name="${name}_right_camera_optical_joint" type="fixed">
+        <origin xyz="0 0 0" rpy="-${M_PI/2} 0.0 -${M_PI/2}"/>
+        <parent link="${name}_right_camera_frame"/>
+        <child link="${name}_right_camera_optical_frame"/>
+      </joint>
+      <!-- ZED2 Sensors -->
+      <xacro:if value="${model == 'zed2'}">
+        <link name="${name}_mag_link" />
+        <joint name="${name}_mag_joint" type="fixed">
+          <parent link="${name}_camera_center"/>
+          <child link="${name}_mag_link"/>
+          <origin xyz="0 0 0" rpy="0 0 0" />
+        </joint>
+        <link name="${name}_baro_link" />
+        <joint name="${name}_baro_joint" type="fixed">
+          <parent link="${name}_camera_center"/>
+          <child link="${name}_baro_link"/>
+          <origin xyz="0 0 0" rpy="0 0 0" />
+        </joint>
+        <link name="${name}_temp_left_link" />
+        <joint name="${name}_temp_left_joint" type="fixed">
+          <parent link="${name}_left_camera_frame"/>
+          <child link="${name}_temp_left_link"/>
+          <origin xyz="0 0 0" rpy="0 0 0" />
+        </joint>
+        <link name="${name}_temp_right_link" />
+        <joint name="${name}_temp_right_joint" type="fixed">
+          <parent link="${name}_right_camera_frame"/>
+          <child link="${name}_temp_right_link"/>
+          <origin xyz="0 0 0" rpy="0 0 0" />
+        </joint>
       </xacro:if>
-    </link>
-    <joint name="${name}_left_camera_joint" type="fixed">
-      <parent link="${name}_camera_center"/>
-      <child link="${name}_left_camera_frame"/>
-      <origin xyz="${optical_offset_x} ${baseline/2} 0" rpy="0 0 0" />
-    </joint>
-    <link name="${name}_left_camera_optical_frame"/>
-    <joint name="${name}_left_camera_optical_joint" type="fixed">
-      <origin xyz="0 0 0" rpy="-${M_PI/2} 0.0 -${M_PI/2}"/>
-      <parent link="${name}_left_camera_frame"/>
-      <child link="${name}_left_camera_optical_frame"/>
-    </joint>
-    <!-- Right Camera -->
-    <link name="${name}_right_camera_frame">
-      <xacro:if value="${model == 'virtual'}">
-        <visual>
-          <origin xyz="0 0 0" rpy="0 0 0"/>
-          <geometry>
-            <mesh filename="package://zed_interfaces/meshes/${model}.stl" />
-          </geometry>
-          <material name="${model}_mat" />
-        </visual>
-        <collision>
-          <origin xyz="0 0 0" rpy="0 0 0"/>
-          <geometry>
-            <mesh filename="package://zed_interfaces/meshes/${model}.stl" />
-          </geometry>
-        </collision>
-      </xacro:if>
-    </link>
-    <joint name="${name}_right_camera_joint" type="fixed">
-      <parent link="${name}_camera_center"/>
-      <child link="${name}_right_camera_frame"/>
-      <origin xyz="${optical_offset_x} -${baseline/2} 0" rpy="0 0 0" />
-    </joint>
-    <link name="${name}_right_camera_optical_frame"/>
-    <joint name="${name}_right_camera_optical_joint" type="fixed">
-      <origin xyz="0 0 0" rpy="-${M_PI/2} 0.0 -${M_PI/2}"/>
-      <parent link="${name}_right_camera_frame"/>
-      <child link="${name}_right_camera_optical_frame"/>
-    </joint>
-    <!-- ZED2 Sensors -->
-    <xacro:if value="${model == 'zed2'}">
-      <link name="${name}_mag_link" />
-      <joint name="${name}_mag_joint" type="fixed">
+    </xacro:unless>
+    <xacro:if value="${mono}">
+      <!-- Camera -->
+      <link name="${name}_camera_frame" />
+      <joint name="${name}_camera_joint" type="fixed">
         <parent link="${name}_camera_center"/>
-        <child link="${name}_mag_link"/>
-        <origin xyz="0 0 0" rpy="0 0 0" />
-      </joint>
-      <link name="${name}_baro_link" />
-      <joint name="${name}_baro_joint" type="fixed">
-        <parent link="${name}_camera_center"/>
-        <child link="${name}_baro_link"/>
-        <origin xyz="0 0 0" rpy="0 0 0" />
-      </joint>
-      <link name="${name}_temp_left_link" />
-      <joint name="${name}_temp_left_joint" type="fixed">
-        <parent link="${name}_left_camera_frame"/>
-        <child link="${name}_temp_left_link"/>
-        <origin xyz="0 0 0" rpy="0 0 0" />
-      </joint>
-      <link name="${name}_temp_right_link" />
-      <joint name="${name}_temp_right_joint" type="fixed">
-        <parent link="${name}_right_camera_frame"/>
-        <child link="${name}_temp_right_link"/>
-        <origin xyz="0 0 0" rpy="0 0 0" />
+        <child link="${name}_camera_frame"/>
+        <origin xyz="${optical_offset_x} 0 0" rpy="0 0 0" />
+      </joint>
+      <link name="${name}_camera_optical_frame"/>
+      <joint name="${name}_camera_optical_joint" type="fixed">
+        <origin xyz="0 0 0" rpy="-${M_PI/2} 0.0 -${M_PI/2}"/>
+        <parent link="${name}_camera_frame"/>
+        <child link="${name}_camera_optical_frame"/>
       </joint>
     </xacro:if>
@@ -194,7 +236,7 @@
       <link name="${name}_gnss_link" />
       <joint name="${name}_gnss_joint" type="fixed">
+        <origin xyz="0 0 0" rpy="0 0 0"/>
         <parent link="${name}_camera_link"/>
         <child link="${name}_gnss_link"/>
-        <xacro:insert_block name="gnss_origin" />
       </joint>
     </xacro:if>
